File: edge/hardware/mdc/generator_load.kicad_sch (KiCad schematic)
At the start: 6 parts, among them M1 Motor_DC, SW1 SW_Rotary_1x4_MP

Commit message: rev3.0 schematics
Connections:
- net at M1.2 (-), R5.1, R6.1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: now also D1.2 (A); no longer D1.1 (K)
- net at M1.1 (+), SW1.5: now also D1.1 (K); no longer D1.2 (A)
Changed lines of the file:
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@@
 	(title_block
 		(title "Generator Load")
-		(date "2026-08-08")
+		(date "2026-08-09")
 		(rev "3.0")
 		(company "Components not part of PCB layout")
@@
 		(exclude_from_sim no)
 		(in_bom yes)
-		(on_board yes)
+		(on_board no)
 		(in_pos_files yes)
 		(dnp no)
@@
 		(lib_id "Device:D")
 		(at 132.08 104.14 90)
+		(mirror x)
 		(unit 1)
 		(body_style 1)
@@
 		(dnp no)
 		(property "Reference" "D1"
-			(at 133.604 103.378 90)
+			(at 133.604 104.902 90)
 			(show_name no)
 			(do_not_autoplace no)
@@
 		)
 		(property "Value" "D"
-			(at 133.604 105.1559 90)
-			(show_name no)
-			(do_not_autoplace no)
+			(at 133.604 103.1241 90)
+			(show_name no)
+			(do_not_autoplace no)

Commit message: finish rev3.0 PCB layout + data collector script changes + firmware changes
Changed lines of the file:
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@@
 			)
 		)
-		(property "Description" "Generator"
+		(property "Description" "DC Motor"
 			(at 118.872 106.68 0)
 			(show_name no)

Commit message: update rev3.0 schematic and layout
Parts:
- removed D1: D, symbol Device:D
Changed lines of the file:
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@@
 	(title_block
 		(title "Generator Load")
-		(date "2026-08-09")
+		(date "2026-08-10")
 		(rev "3.0")
 		(company "Components not part of PCB layout")
@@
 	)
 	(junction
-		(at 132.08 110.49)
-		(diameter 0)
-		(color 0 0 0 0)
-	)
-	(junction
 		(at 167.64 97.79)
 		(diameter 0)
 		(color 0 0 0 0)
 	)
-	(junction
-		(at 132.08 97.79)
-		(diameter 0)
-		(color 0 0 0 0)
-	)
 	(no_connect
 		(at 153.67 92.71)
@@
 	(wire
 		(pts
-			(xy 123.19 97.79) (xy 132.08 97.79)
-		)
-		(stroke
-			(width 0)
-			(type default)
-		)
-	)
-	(wire
-		(pts
-			(xy 132.08 107.95) (xy 132.08 110.49)
+			(xy 123.19 97.79) (xy 138.43 97.79)
 		)
 		(stroke
@@
 	(wire
 		(pts
-			(xy 123.19 110.49) (xy 132.08 110.49)
-		)
-		(stroke
-			(width 0)
-			(type default)
-		)
-	)
-	(wire
-		(pts
-			(xy 132.08 110.49) (xy 167.64 110.49)
-		)
-		(stroke
-			(width 0)
-			(type default)
-		)
-	)
-	(wire
-		(pts
-			(xy 132.08 97.79) (xy 138.43 97.79)
+			(xy 123.19 110.49) (xy 167.64 110.49)
 		)
 		(stroke
@@
 		(pts
 			(xy 165.1 95.25) (xy 167.64 95.25)
-		)
-		(stroke
-			(width 0)
-			(type default)
-		)
-	)
-	(wire
-		(pts
-			(xy 132.08 97.79) (xy 132.08 100.33)
 		)
 		(stroke
@@
 					(unit 1)
 				)
-			)
-		)
-	)
-	(symbol
-		(lib_id "Device:D")
-		(at 132.08 104.14 90)
-		(mirror x)
-		(unit 1)
-		(body_style 1)
-		(exclude_from_sim no)
-		(in_bom yes)
-		(on_board no)
-		(in_pos_files yes)
-		(dnp no)
-		(property "Reference" "D1"
-			(at 133.604 104.902 90)
-			(show_name no)
-			(do_not_autoplace no)
-			(effects
-				(font
-					(size 1.27 1.27)
-				)
-				(justify right)
-			)
-		)
-		(property "Value" "D"
-			(at 133.604 103.1241 90)
-			(show_name no)
-			(do_not_autoplace no)
-			(effects
-				(font
-					(size 1.27 1.27)
-				)
-				(justify right)
-			)
-		)
-		(property "Footprint" ""
-			(at 132.08 104.14 0)
-			(hide yes)
-			(show_name no)
-			(do_not_autoplace no)
-			(effects
-				(font
-					(size 1.27 1.27)
-				)
-			)
-		)
-		(property "Datasheet" ""
-			(at 132.08 104.14 0)
-			(hide yes)
-			(show_name no)
-			(do_not_autoplace no)
-			(effects
-				(font
-					(size 1.27 1.27)
-				)
-			)
-		)
-		(property "Description" "Diode"
-			(at 132.08 104.14 0)
-			(hide yes)
-			(show_name no)
-			(do_not_autoplace no)
-			(effects
-				(font
-					(size 1.27 1.27)
-				)
-			)
-		)
-		(property "Sim.Device" "D"
-			(at 132.08 104.14 0)
-			(hide yes)
-			(show_name no)
-			(do_not_autoplace no)
-			(effects
-				(font
-					(size 1.27 1.27)
-				)
-			)
-		)
-		(property "Sim.Pins" "1=K 2=A"
-			(at 132.08 104.14 0)
-			(hide yes)
-			(show_name no)
-			(do_not_autoplace no)
-			(effects
-				(font
-					(size 1.27 1.27)
-				)
-			)
-		)
-		(pin "1"
-		)
-		(pin "2"
-		)
-		(instances
-			(project "mdc"
-				(path "/813130ed-0e1e-452d-b14e-fae57783a961/7a2822f0-8a73-4068-9237-8ac59dd9220e"
-					(reference "D1")
-					(unit 1)
-				)
