File: edge/hardware/mdc/microcontroller.kicad_sch (KiCad schematic)
At the start: 1 part, among them U1 ESP32-S3-DEVKITC-1-N16R8V

Commit message: finish rev3.0 PCB layout + data collector script changes + firmware changes
Parts:
- U1: footprint Espressif:ESP32-S3-DevKitC -> ESP32-S3-DEVKITC-1-N16R8V:XCVR_ESP32-S3-DEVKITC-1-N16R8V
Connections:
- net +3V3: now also U1.J1_1 (3V3), U1.J1_2 (3V3); no longer U1.1 (3V3), U1.2 (3V3)
- net GND: now also U1.J1_22 (GND), U1.J3_1 (GND), U1.J3_21 (GND), U1.J3_22 (GND); no longer U1.22 (GND), U1.23 (GND), U1.24 (GND), U1.44 (GND)
- net GPIO38: now also U1.J3_10 (GPIO38); no longer U1.35 (GPIO38)
- net GPIO39: now also U1.J3_9 (MTCK/GPIO39); no longer U1.36 (MTCK/GPIO39)
- net GPIO40: now also U1.J3_8 (MTDO/GPIO40); no longer U1.37 (MTDO/GPIO40)
- net GPIO41: now also U1.J3_7 (MTDI/GPIO41); no longer U1.38 (MTDI/GPIO41)
- net I2C_SCL: now also U1.J1_4 (GPIO4); no longer U1.4 (GPIO4)
- net I2C_SDA: now also U1.J1_5 (GPIO5); no longer U1.5 (GPIO5)
- net I2S_SCK: now also U1.J1_10 (GPIO17); no longer U1.10 (GPIO17)
- net I2S_SD: now also U1.J1_11 (GPIO18); no longer U1.11 (GPIO18)
- net I2S_WS: now also U1.J1_9 (GPIO16); no longer U1.9 (GPIO16)
- net SPI_CS: now also U1.J1_19 (GPIO13); no longer U1.19 (GPIO13)
- net SPI_SCL: now also U1.J1_18 (GPIO12); no longer U1.18 (GPIO12)
- net SPI_SDA: now also U1.J1_17 (GPIO11); no longer U1.17 (GPIO11)
- net SPI_SDO: now also U1.J1_16 (GPIO10); no longer U1.16 (GPIO10)
- new net ISENSE: U1.J1_7 (GPIO7)
- no-connect marks 25 -> 24
Changed lines of the file:
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@@
-	)
-	(no_connect
-		(at 118.11 97.79)
 	)
 	(no_connect
@@
 		(pts
 			(xy 115.57 123.19) (xy 118.11 123.19)
+		)
+		(stroke
+			(width 0)
+			(type default)
+		)
+	)
+	(wire
+		(pts
+			(xy 115.57 97.79) (xy 118.11 97.79)
 		)
 		(stroke
@@
 		(property "Intersheetrefs" "${INTERSHEET_REFS}"
 			(at 104.7229 105.41 0)
+			(hide yes)
+			(show_name no)
+			(do_not_autoplace no)
+			(effects
+				(font
+					(size 1.27 1.27)
+				)
+				(justify right)
+			)
+		)
+	)
+	(global_label "ISENSE"
+		(shape input)
+		(at 115.57 97.79 180)
+		(fields_autoplaced yes)
+		(effects
+			(font
+				(size 1.27 1.27)
+			)
+			(justify right)
+		)
+		(property "Intersheetrefs" "${INTERSHEET_REFS}"
+			(at 105.9325 97.79 0)
 			(hide yes)
 			(show_name no)
@@
 			)
 		)
-		(property "Footprint" "Espressif:ESP32-S3-DevKitC"
+		(property "Footprint" "ESP32-S3-DEVKITC-1-N16R8V:XCVR_ESP32-S3-DEVKITC-1-N16R8V"
 			(at 140.97 100.33 0)
 			(hide yes)
@@
 			)
 		)
-		(pin "40"
-		)
-		(pin "38"
-		)
-		(pin "33"
-		)
-		(pin "23"
-		)
-		(pin "28"
-		)
-		(pin "36"
-		)
-		(pin "35"
-		)
-		(pin "31"
-		)
-		(pin "25"
-		)
-		(pin "26"
-		)
-		(pin "29"
-		)
-		(pin "1"
-		)
-		(pin "3"
-		)
-		(pin "34"
-		)
-		(pin "2"
-		)
-		(pin "32"
-		)
-		(pin "27"
-		)
-		(pin "30"
-		)
-		(pin "5"
-		)
-		(pin "41"
-		)
-		(pin "16"
-		)
-		(pin "20"
-		)
-		(pin "12"
-		)
-		(pin "39"
-		)
-		(pin "8"
-		)
-		(pin "21"
-		)
-		(pin "17"
-		)
-		(pin "22"
-		)
-		(pin "7"
-		)
-		(pin "13"
-		)
-		(pin "43"
-		)
-		(pin "37"
-		)
-		(pin "11"
-		)
-		(pin "6"
-		)
-		(pin "19"
-		)
-		(pin "15"
-		)
-		(pin "9"
-		)
-		(pin "10"
-		)
-		(pin "14"
-		)
-		(pin "42"
-		)
-		(pin "24"
-		)
-		(pin "44"
-		)
-		(pin "4"
-		)
-		(pin "18"
+		(pin "J1_16"
+		)
+		(pin "J1_12"
+		)
+		(pin "J1_4"
+		)
+		(pin "J1_14"
+		)
+		(pin "J1_6"
+		)
+		(pin "J1_5"
+		)
+		(pin "J1_11"
+		)
+		(pin "J1_10"
+		)
+		(pin "J1_13"
+		)
+		(pin "J1_2"
+		)
+		(pin "J1_7"
+		)
+		(pin "J1_1"
+		)
+		(pin "J1_18"
+		)
+		(pin "J1_3"
+		)
+		(pin "J1_9"
+		)
+		(pin "J1_15"
+		)
+		(pin "J1_8"
+		)
+		(pin "J1_17"
+		)
+		(pin "J1_21"
+		)
+		(pin "J3_19"
+		)
+		(pin "J1_22"
+		)
+		(pin "J3_18"
+		)
+		(pin "J3_4"
+		)
+		(pin "J3_14"
+		)
+		(pin "J3_13"
+		)
+		(pin "J3_16"
+		)
+		(pin "J3_5"
+		)
+		(pin "J3_2"
+		)
+		(pin "J3_10"
+		)
+		(pin "J3_21"
+		)
+		(pin "J3_9"
+		)
+		(pin "J3_8"
+		)
+		(pin "J3_3"
+		)
+		(pin "J1_20"
+		)
+		(pin "J3_11"
+		)
+		(pin "J1_19"
+		)
+		(pin "J3_7"
+		)
+		(pin "J3_1"
+		)
+		(pin "J3_22"
+		)
+		(pin "J3_6"
+		)
+		(pin "J3_20"
+		)
+		(pin "J3_12"
+		)
+		(pin "J3_17"
+		)
+		(pin "J3_15"
 		)
 		(instances

Commit message: update rev3.0 schematic and layout
Parts:
- added C4: 100nF, Capacitor_THT:C_Disc_D5.0mm_W2.5mm_P5.00mm, symbol Device:C_Small
- added C5: 10uF 16V, Capacitor_THT:CP_Radial_D5.0mm_P2.50mm, symbol Device:C_Polarized_Small
Connections:
- net +3V3: now also C4.2, C5.1
- net GND: now also C4.1, C5.2
