File: edge/hardware/mdc/motor_driver.kicad_sch (KiCad schematic)
At the start: 10 parts, among them J1 Conn_01x06, Q1 2N7000, Q2 2N7000, Q3 2N7000, Q4 2N7000, U5 74HC04

Commit message: rev3.0 schematics
Parts:
- added C1: 100nF, symbol Device:C_Small
- added R10, R11, R8, R9: 100K, symbol Device:R_Small
- added unit 5 of U5
- added unit 6 of U5
Connections:
- net +5V: now also C1.1
- net GND: now also C1.2, R10.2, R11.2, R8.2, R9.2, U5.11, U5.13
- net GPIO38: now also R11.1
- net GPIO39: now also R10.1
- net GPIO40: now also R9.1
- net GPIO41: now also R8.1
- no-connect marks 0 -> 2
Other:
- moved on the sheet: J1, Q1, Q2, Q3, Q4, R1, R2, R3, R4, U5A, U5B, U5C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

Commit message: finish rev3.0 PCB layout + data collector script changes + firmware changes
Parts:
- C1: footprint (none) -> Capacitor_THT:C_Disc_D5.0mm_W2.5mm_P5.00mm
- R1, R2, R3, R4: value 10K -> 10k; footprint Resistor_THT:R_Axial_DIN0207_L6.3mm_D2.5mm_P10.16mm_Horizontal -> Resistor_THT:R_Axial_DIN0207_L6.3mm_D2.5mm_P7.62mm_Horizontal
- R10, R11, R8, R9: value 100K -> 100k; footprint (none) -> Resistor_THT:R_Axial_DIN0207_L6.3mm_D2.5mm_P7.62mm_Horizontal
- U5: footprint (none) -> Package_DIP:DIP-14_W7.62mm

Commit message: update rev3.0 schematic and layout
Parts:
- R1, R2, R3, R4: value 10k -> 2.2k
Connections:
- net GND: now also U5.10, U5.12; no longer U5.11, U5.13
Other:
- moved on the sheet: U5E, U5F

Commit message: update rev3.0 schematic and layout
Connections:
- net GND: now also U5.11, U5.13; no longer U5.10, U5.12
Other:
- moved on the sheet: U5E, U5F
Changed lines of the file:
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@@
 	(title_block
 		(title "Motor Driver")
-		(date "2026-08-10")
+		(date "2026-08-11")
 		(rev "3.0")
 		(comment 1 "Department of EECS- AIoT and Energy Management Lab")
@@
 	)
 	(no_connect
-		(at 59.69 144.78)
+		(at 44.45 137.16)
 	)
 	(no_connect
-		(at 36.83 144.78)
+		(at 64.77 137.16)
 	)
 	(wire
@@
 	(wire
 		(pts
-			(xy 74.93 144.78) (xy 74.93 147.32)
-		)
-		(stroke
-			(width 0)
-			(type default)
-		)
-	)
-	(wire
-		(pts
 			(xy 238.76 77.47) (xy 238.76 76.2)
 		)
@@
 	(wire
 		(pts
-			(xy 52.07 144.78) (xy 52.07 147.32)
-		)
-		(stroke
-			(width 0)
-			(type default)
-		)
-	)
-	(wire
-		(pts
 			(xy 132.08 63.5) (xy 132.08 66.04)
 		)
@@
 	(symbol
 		(lib_id "74xx:74HC04")
-		(at 44.45 144.78 0)
+		(at 44.45 144.78 90)
 		(unit 5)
 		(body_style 1)
@@
 		(fields_autoplaced yes)
 		(property "Reference" "U5"
-			(at 44.45 135.89 0)
+			(at 49.53 143.5099 90)
 			(show_name no)
 			(do_not_autoplace no)
@@
 					(size 1.27 1.27)
 				)
+				(justify right)
 			)
 		)
 		(property "Value" "74HC04"
-			(at 44.45 138.43 0)
+			(at 49.53 146.0499 90)
 			(show_name no)
 			(do_not_autoplace no)
@@
 					(size 1.27 1.27)
 				)
+				(justify right)
 			)
 		)
@@
 	)
 	(symbol
-		(lib_id "power:GND")
-		(at 52.07 147.32 0)
-		(unit 1)
-		(body_style 1)
-		(exclude_from_sim no)
-		(in_bom yes)
-		(on_board yes)
-		(in_pos_files yes)
-		(dnp no)
-		(fields_autoplaced yes)
-		(property "Reference" "#PWR025"
-			(at 52.07 153.67 0)
-			(hide yes)
-			(show_name no)
-			(do_not_autoplace no)
-			(effects
-				(font
-					(size 1.27 1.27)
-				)
-			)
-		)
-		(property "Value" "GND"
-			(at 52.07 152.4 0)
-			(show_name no)
-			(do_not_autoplace no)
-			(effects
-				(font
-					(size 1.27 1.27)
-				)
-			)
-		)
-		(property "Footprint" ""
-			(at 52.07 147.32 0)
-			(hide yes)
-			(show_name no)
-			(do_not_autoplace no)
-			(effects
-				(font
-					(size 1.27 1.27)
-				)
-			)
-		)
-		(property "Datasheet" ""
-			(at 52.07 147.32 0)
-			(hide yes)
-			(show_name no)
-			(do_not_autoplace no)
-			(effects
-				(font
-					(size 1.27 1.27)
-				)
-			)
-		)
-		(property "Description" "Power symbol creates a global label with name \"GND\" , ground"
-			(at 52.07 147.32 0)
-			(hide yes)
-			(show_name no)
-			(do_not_autoplace no)
-			(effects
-				(font
-					(size 1.27 1.27)
-				)
-			)
-		)
-		(pin "1"
-		)
-		(instances
-			(project "mdc"
-				(path "/813130ed-0e1e-452d-b14e-fae57783a961/8f2924e4-fc6a-4bbc-8379-4544cedaebc8"
-					(reference "#PWR025")
-					(unit 1)
-				)
-			)
-		)
-	)
-	(symbol
 		(lib_id "Device:C_Small")
 		(at 90.17 144.78 0)
@@
 	)
 	(symbol
+		(lib_id "power:GND")
+		(at 44.45 152.4 0)
+		(unit 1)
+		(body_style 1)
+		(exclude_from_sim no)
+		(in_bom yes)
+		(on_board yes)
+		(in_pos_files yes)
+		(dnp no)
+		(fields_autoplaced yes)
+		(property "Reference" "#PWR025"
+			(at 44.45 158.75 0)
+			(hide yes)
+			(show_name no)
+			(do_not_autoplace no)
+			(effects
+				(font
+					(size 1.27 1.27)
+				)
+			)
+		)
+		(property "Value" "GND"
+			(at 44.45 157.48 0)
+			(show_name no)
+			(do_not_autoplace no)
+			(effects
+				(font
+					(size 1.27 1.27)
+				)
+			)
+		)
+		(property "Footprint" ""
+			(at 44.45 152.4 0)
+			(hide yes)
+			(show_name no)
+			(do_not_autoplace no)
+			(effects
+				(font
+					(size 1.27 1.27)
+				)
+			)
+		)
+		(property "Datasheet" ""
+			(at 44.45 152.4 0)
+			(hide yes)
+			(show_name no)
+			(do_not_autoplace no)
+			(effects
+				(font
+					(size 1.27 1.27)
+				)
+			)
+		)
+		(property "Description" "Power symbol creates a global label with name \"GND\" , ground"
+			(at 44.45 152.4 0)
+			(hide yes)
+			(show_name no)
+			(do_not_autoplace no)
+			(effects
+				(font
+					(size 1.27 1.27)
+				)
+			)
+		)
+		(pin "1"
+		)
+		(instances
+			(project "mdc"
+				(path "/813130ed-0e1e-452d-b14e-fae57783a961/8f2924e4-fc6a-4bbc-8379-4544cedaebc8"
+					(reference "#PWR025")
+					(unit 1)
+				)
+			)
+		)
+	)
+	(symbol
 		(lib_id "74xx:74HC04")
 		(at 99.06 144.78 0)
@@
 	(symbol
 		(lib_id "power:GND")
+		(at 64.77 152.4 0)
+		(unit 1)
+		(body_style 1)
+		(exclude_from_sim no)
+		(in_bom yes)
+		(on_board yes)
+		(in_pos_files yes)
+		(dnp no)
+		(fields_autoplaced yes)
+		(property "Reference" "#PWR026"
+			(at 64.77 158.75 0)
+			(hide yes)
+			(show_name no)
+			(do_not_autoplace no)
+			(effects
+				(font
+					(size 1.27 1.27)
+				)
+			)
+		)
+		(property "Value" "GND"
+			(at 64.77 157.48 0)
+			(show_name no)
+			(do_not_autoplace no)
+			(effects
+				(font
+					(size 1.27 1.27)
+				)
+			)
+		)
+		(property "Footprint" ""
+			(at 64.77 152.4 0)
+			(hide yes)
+			(show_name no)
+			(do_not_autoplace no)
+			(effects
+				(font
+					(size 1.27 1.27)
+				)
+			)
+		)
+		(property "Datasheet" ""
+			(at 64.77 152.4 0)
+			(hide yes)
+			(show_name no)
+			(do_not_autoplace no)
+			(effects
+				(font
+					(size 1.27 1.27)
+				)
+			)
+		)
+		(property "Description" "Power symbol creates a global label with name \"GND\" , ground"
+			(at 64.77 152.4 0)
+			(hide yes)
+			(show_name no)
+			(do_not_autoplace no)
+			(effects
+				(font
+					(size 1.27 1.27)
+				)
+			)
+		)
+		(pin "1"
+		)
+		(instances
+			(project "mdc"
+				(path "/813130ed-0e1e-452d-b14e-fae57783a961/8f2924e4-fc6a-4bbc-8379-4544cedaebc8"
+					(reference "#PWR026")
+					(unit 1)
+				)
+			)
+		)
+	)
+	(symbol
+		(lib_id "power:GND")
 		(at 99.06 157.48 0)
 		(unit 1)
@@
 	(symbol
 		(lib_id "74xx:74HC04")
-		(at 67.31 144.78 0)
+		(at 64.77 144.78 90)
 		(unit 6)
 		(body_style 1)
@@
 		(fields_autoplaced yes)
 		(property "Reference" "U5"
-			(at 67.31 135.89 0)
+			(at 69.85 143.5099 90)
 			(show_name no)
 			(do_not_autoplace no)
@@
 					(size 1.27 1.27)
 				)
+				(justify right)
 			)
 		)
 		(property "Value" "74HC04"
-			(at 67.31 138.43 0)
+			(at 69.85 146.0499 90)
 			(show_name no)
 			(do_not_autoplace no)
@@
 					(size 1.27 1.27)
 				)
+				(justify right)
 			)
 		)
 		(property "Footprint" "Package_DIP:DIP-14_W7.62mm"
-			(at 67.31 144.78 0)
+			(at 64.77 144.78 0)
 			(hide yes)
 			(show_name no)
@@
 		)
 		(property "Datasheet" "https://assets.nexperia.com/documents/data-sheet/74HC_HCT04.pdf"
-			(at 67.31 144.78 0)
+			(at 64.77 144.78 0)
 			(hide yes)
 			(show_name no)
@@
 		)
 		(property "Description" "Hex Inverter"
-			(at 67.31 144.78 0)
+			(at 64.77 144.78 0)
 			(hide yes)
 			(show_name no)
@@
 					(unit 1)
 				)
-			)
-		)
-	)
-	(symbol
-		(lib_id "power:GND")
-		(at 74.93 147.32 0)
-		(unit 1)
-		(body_style 1)
-		(exclude_from_sim no)
-		(in_bom yes)
-		(on_board yes)
-		(in_pos_files yes)
-		(dnp no)
-		(fields_autoplaced yes)
-		(property "Reference" "#PWR026"
-			(at 74.93 153.67 0)
-			(hide yes)
-			(show_name no)
-			(do_not_autoplace no)
-			(effects
-				(font
-					(size 1.27 1.27)
-				)
-			)
-		)
-		(property "Value" "GND"
-			(at 74.93 152.4 0)
-			(show_name no)
-			(do_not_autoplace no)
-			(effects
-				(font
-					(size 1.27 1.27)
-				)
-			)
-		)
-		(property "Footprint" ""
-			(at 74.93 147.32 0)
-			(hide yes)
-			(show_name no)
-			(do_not_autoplace no)
-			(effects
-				(font
-					(size 1.27 1.27)
-				)
-			)
-		)
-		(property "Datasheet" ""
-			(at 74.93 147.32 0)
-			(hide yes)
-			(show_name no)
-			(do_not_autoplace no)
-			(effects
-				(font
-					(size 1.27 1.27)
-				)
-			)
-		)
-		(property "Description" "Power symbol creates a global label with name \"GND\" , ground"
-			(at 74.93 147.32 0)
-			(hide yes)
-			(show_name no)
-			(do_not_autoplace no)
-			(effects
-				(font
-					(size 1.27 1.27)
-				)
-			)
-		)
-		(pin "1"
-		)
-		(instances
-			(project "mdc"
-				(path "/813130ed-0e1e-452d-b14e-fae57783a961/8f2924e4-fc6a-4bbc-8379-4544cedaebc8"
-					(reference "#PWR026")
-					(unit 1)
-				)
